File: Projects/ZeusAmp/ZeusAmp.sch (KiCad schematic (older format))
At the start: 74 parts, among them Q1 NZT660, Q11 NZT660, Q12 NZT660, Q121 NZT660, Q2 NZT660, Q21 NZT660, Q3 PZTA06, Q31 PZTA06, Q4 MJD340T4, Q41 MJD340T4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

Commit message: Added Drill holes
Parts:
- added H1, H2, H3, H4: MountingHole_Pad, MountingHole:MountingHole_2.2mm_M2, symbol Mechanical:MountingHole_Pad
Connections:
- net GND: now also H1.1, H2.1, H3.1, H4.1
Changed lines of the file:
@@
 Wire Wire Line
 	13425 1225 13200 1225
+$Comp
+L Mechanical:MountingHole_Pad H1
+U 1 1 604B9952
+P 12525 3350
+F 0 "H1" H 12625 3399 50  0000 L CNN
+F 1 "MountingHole_Pad" H 12625 3308 50  0000 L CNN
+F 2 "MountingHole:MountingHole_2.2mm_M2" H 12525 3350 50  0001 C CNN
+F 3 "~" H 12525 3350 50  0001 C CNN
+	1    12525 3350
+	1    0    0    -1
+$EndComp
+$Comp
+L power:GND #PWR?
+U 1 1 604B9CD2
+P 12525 3450
+F 0 "#PWR?" H 12525 3200 50  0001 C CNN
+F 1 "GND" H 12530 3277 50  0000 C CNN
+F 2 "" H 12525 3450 50  0001 C CNN
+F 3 "" H 12525 3450 50  0001 C CNN
+	1    12525 3450
+	1    0    0    -1
+$EndComp
+$Comp
+L Mechanical:MountingHole_Pad H2
+U 1 1 604C84EB
+P 13700 3325
+F 0 "H2" H 13800 3374 50  0000 L CNN
+F 1 "MountingHole_Pad" H 13800 3283 50  0000 L CNN
+F 2 "MountingHole:MountingHole_2.2mm_M2" H 13700 3325 50  0001 C CNN
+F 3 "~" H 13700 3325 50  0001 C CNN
+	1    13700 3325
+	1    0    0    -1
+$EndComp
+$Comp
+L power:GND #PWR?
+U 1 1 604C84F1
+P 13700 3425
+F 0 "#PWR?" H 13700 3175 50  0001 C CNN
+F 1 "GND" H 13705 3252 50  0000 C CNN
+F 2 "" H 13700 3425 50  0001 C CNN
+F 3 "" H 13700 3425 50  0001 C CNN
+	1    13700 3425
+	1    0    0    -1
+$EndComp
+$Comp
+L Mechanical:MountingHole_Pad H3
+U 1 1 604D53CF
+P 12500 3900
+F 0 "H3" H 12600 3949 50  0000 L CNN
+F 1 "MountingHole_Pad" H 12600 3858 50  0000 L CNN
+F 2 "MountingHole:MountingHole_2.2mm_M2" H 12500 3900 50  0001 C CNN
+F 3 "~" H 12500 3900 50  0001 C CNN
+	1    12500 3900
+	1    0    0    -1
+$EndComp
+$Comp
+L power:GND #PWR?
+U 1 1 604D53D5
+P 12500 4000
+F 0 "#PWR?" H 12500 3750 50  0001 C CNN
+F 1 "GND" H 12505 3827 50  0000 C CNN
+F 2 "" H 12500 4000 50  0001 C CNN
+F 3 "" H 12500 4000 50  0001 C CNN
+	1    12500 4000
+	1    0    0    -1
+$EndComp
+$Comp
+L Mechanical:MountingHole_Pad H4
+U 1 1 604D53DB
+P 13675 3875
+F 0 "H4" H 13775 3924 50  0000 L CNN
+F 1 "MountingHole_Pad" H 13775 3833 50  0000 L CNN
+F 2 "MountingHole:MountingHole_2.2mm_M2" H 13675 3875 50  0001 C CNN
+F 3 "~" H 13675 3875 50  0001 C CNN
+	1    13675 3875
+	1    0    0    -1
+$EndComp
+$Comp
+L power:GND #PWR?
+U 1 1 604D53E1
+P 13675 3975
+F 0 "#PWR?" H 13675 3725 50  0001 C CNN
+F 1 "GND" H 13680 3802 50  0000 C CNN
+F 2 "" H 13675 3975 50  0001 C CNN
+F 3 "" H 13675 3975 50  0001 C CNN
+	1    13675 3975
+	1    0    0    -1
+$EndComp
 $EndSCHEMATC

Commit message: added switch
Parts:
- added S1: 100SP1T1B4M2QE, SW_100SP1T1B4M2QE, symbol 100SP1T1B4M2QE:100SP1T1B4M2QE
Connections:
- net V+: now also S1.2; no longer 16VACIn1.1
- new net: 16VACIn1.1, S1.1
- no-connect marks 0 -> 1
Other:
- moved on the sheet: 16VACIn1
Changed lines of the file:
@@
 L Connector:Barrel_Jack 16VACIn1
 U 1 1 604DBD92
-P 13925 1325
-F 0 "16VACIn1" H 13695 1375 50  0000 R CNN
-F 1 "Barrel_Jack" H 13695 1284 50  0000 R CNN
-F 2 "Connector_BarrelJack:BarrelJack_Horizontal" H 13975 1285 50  0001 C CNN
-F 3 "~" H 13975 1285 50  0001 C CNN
-	1    13925 1325
+P 14850 1275
+F 0 "16VACIn1" H 14620 1325 50  0000 R CNN
+F 1 "Barrel_Jack" H 14620 1234 50  0000 R CNN
+F 2 "Connector_BarrelJack:BarrelJack_Horizontal" H 14900 1235 50  0001 C CNN
+F 3 "~" H 14900 1235 50  0001 C CNN
+	1    14850 1275
 	-1   0    0    -1
 $EndComp
@@
 L power:GND #PWR?
 U 1 1 604C2102
-P 13625 1425
-F 0 "#PWR?" H 13625 1175 50  0001 C CNN
-F 1 "GND" H 13630 1252 50  0000 C CNN
-F 2 "" H 13625 1425 50  0001 C CNN
-F 3 "" H 13625 1425 50  0001 C CNN
-	1    13625 1425
+P 14550 1375
+F 0 "#PWR?" H 14550 1125 50  0001 C CNN
+F 1 "GND" H 14555 1202 50  0000 C CNN
+F 2 "" H 14550 1375 50  0001 C CNN
+F 3 "" H 14550 1375 50  0001 C CNN
+	1    14550 1375
 	1    0    0    -1
 $EndComp
@@
 	1    0    0    -1
 $EndComp
+NoConn ~ 14225 1325
+$Comp
+L 100SP1T1B4M2QE:100SP1T1B4M2QE S1
+U 1 1 6050C042
+P 13925 1225
+F 0 "S1" H 13925 1506 50  0000 C CNN
+F 1 "100SP1T1B4M2QE" H 13925 1415 50  0000 C CNN
+F 2 "SW_100SP1T1B4M2QE" H 13925 1225 50  0001 L BNN
+F 3 "" H 13925 1225 50  0001 L BNN
+F 4 "E" H 13925 1225 50  0001 L BNN "PARTREV"
+F 5 "E-Switch" H 13925 1225 50  0001 L BNN "MANUFACTURER"
+F 6 "29.68 mm" H 13925 1225 50  0001 L BNN "MAXIMUM_PACKAGE_HEIGHT"
+F 7 "Manufacturer Recommendations" H 13925 1225 50  0001 L BNN "STANDARD"
+	1    13925 1225
+	1    0    0    -1
+$EndComp
+Wire Wire Line
+	14225 1125 14550 1125
+Wire Wire Line
+	14550 1125 14550 1175
 $EndSCHEMATC
